Commit message: added urdf and instance files for forearm working like turbodrivers testing

File: instance/instances/robots/xacro/mechanisms/mechanisms.xacro (robot description, xacro)
@@ -33,3 +33,12 @@
     </Mechanism>
 </xacro:macro>
+<xacro:macro name="forearm_new_firmware_mechanism" params="prefix forearm_j1_serial_number forearm_j2_serial_number forearm_j3_serial_number forearm_j4_serial_number forearm_j5_serial_number forearm_j6_serial_number wrist_bottom_serial_number wrist_top_serial_number">
+	<xacro:simple_mechanism name="${IndexFingerPitch1JointName}" serial_number="${forearm_j1_serial_number}" node="${IndexFingerPitch1Node}"/>
+	<xacro:simple_mechanism name="${MiddleFingerPitch1JointName}" serial_number="${forearm_j2_serial_number}" node="${MiddleFingerPitch1Node}"/>
+	<xacro:simple_mechanism name="${PinkyPitch1JointName}" serial_number="${forearm_j3_serial_number}" node="${PinkyPitch1Node}"/>
+	<xacro:simple_mechanism name="${ThumbRollJointName}" serial_number="${forearm_j4_serial_number}" node="${ThumbRollNode}"/>
+	<xacro:simple_mechanism name="${ThumbPitch1JointName}" serial_number="${forearm_j5_serial_number}" node="${ThumbPitch1Node}"/>
+	<xacro:simple_mechanism name="${ThumbPitch2JointName}" serial_number="${forearm_j6_serial_number}" node="${ThumbPitch2Node}"/>
+	<xacro:two_active_joint_mechanism mechanism_name="${prefix}Wrist" actuator0_name="${WristBottomActuatorName}" actuator1_name="${WristTopActuatorName}" joint0_name="${WristRollJointName}" joint1_name="${WristPitchJointName}" actuator0_serial="${wrist_bottom_serial_number}" actuator1_serial="${wrist_top_serial_number}" actuator0_node="${WristBottomActuatorNode}" actuator1_node="${WristTopActuatorNode}" />
+</xacro:macro>
 </robot>

File: model/robots/common/xacro/arm/arm.xacro (robot description, xacro)
@@ -3,5 +3,4 @@
   <xacro:include filename="$(find val_description)/common/xacro/joint_names/valkyrie_joint_names.xacro"/>
   <xacro:include filename="$(find val_description)/common/xacro/actuator_names/valkyrie_actuator_names.xacro"/>
-  <xacro:include filename="$(find val_description)/common/xacro/nodes/valkyrie_nodes.xacro"/>
   <xacro:include filename="$(find val_description)/model/robots/common/xacro/arm/joint_axes.xacro"/>
   <xacro:include filename="$(find val_description)/model/robots/common/xacro/arm/link_names.xacro"/>

File: model/robots/common/xacro/head/head.xacro (robot description, xacro)
@@ -2,5 +2,4 @@
   <xacro:include filename="$(find val_description)/common/xacro/joint_names/valkyrie_joint_names.xacro"/>
   <xacro:include filename="$(find val_description)/common/xacro/actuator_names/valkyrie_actuator_names.xacro"/>
-  <xacro:include filename="$(find val_description)/common/xacro/nodes/valkyrie_nodes.xacro"/>
   <xacro:include filename="$(find val_description)/model/robots/common/xacro/head/joint_axes.xacro"/>
   <xacro:include filename="$(find val_description)/model/robots/common/xacro/head/link_names.xacro"/>

File: model/robots/common/xacro/leg/leg.xacro (robot description, xacro)
@@ -3,5 +3,4 @@
   <xacro:include filename="$(find val_description)/common/xacro/joint_names/valkyrie_joint_names.xacro"/>
   <xacro:include filename="$(find val_description)/common/xacro/actuator_names/valkyrie_actuator_names.xacro"/>
-  <xacro:include filename="$(find val_description)/common/xacro/nodes/valkyrie_nodes.xacro"/>
   <xacro:include filename="$(find val_description)/model/robots/common/xacro/leg/joint_axes.xacro"/>
   <xacro:include filename="$(find val_description)/model/robots/common/xacro/leg/link_names.xacro"/>

File: model/robots/common/xacro/waist/waist.xacro (robot description, xacro)
@@ -2,5 +2,4 @@
   <xacro:include filename="$(find val_description)/common/xacro/joint_names/valkyrie_joint_names.xacro"/>
   <xacro:include filename="$(find val_description)/common/xacro/actuator_names/valkyrie_actuator_names.xacro"/>
-  <xacro:include filename="$(find val_description)/common/xacro/nodes/valkyrie_nodes.xacro"/>
   <xacro:include filename="$(find val_description)/model/robots/common/xacro/waist/joint_axes.xacro"/>
   <xacro:include filename="$(find val_description)/model/robots/common/xacro/waist/joint_axes.xacro"/>

File: model/robots/forearm_left.xacro (robot description, xacro)
@@ -4,4 +4,5 @@
     <xacro:include filename="$(find val_description)/model/robots/common/xacro/common_bodies.xacro" />
     <xacro:include filename="$(find val_description)/common/xacro/api/forearm_api.xacro"/>
+    <xacro:include filename="$(find val_description)/common/xacro/nodes/valkyrie_nodes.xacro"/>
     <xacro:property name="prefix" value="left"/>
     <xacro:property name="reflect" value="1"/>

File: model/robots/forearm_right.xacro (robot description, xacro)
@@ -4,4 +4,5 @@
     <xacro:include filename="$(find val_description)/model/robots/common/xacro/common_bodies.xacro" />
     <xacro:include filename="$(find val_description)/common/xacro/api/forearm_api.xacro"/>
+    <xacro:include filename="$(find val_description)/common/xacro/nodes/valkyrie_nodes.xacro"/>
     <xacro:property name="prefix" value="right"/>
     <xacro:property name="reflect" value="-1"/>

File: model/robots/imu_test.xacro (robot description, xacro)
@@ -4,4 +4,5 @@
     <xacro:include filename="$(find val_description)/model/robots/common/xacro/common_bodies.xacro" />
     <xacro:include filename="$(find val_description)/model/robots/common/xacro/valkyrie_imu_base.xacro"/>
+    <xacro:include filename="$(find val_description)/common/xacro/nodes/valkyrie_nodes.xacro"/>
     <xacro:include filename="$(find val_description)/common/xacro/serial_numbers/valkyrie_C_serials.xacro"/>
     <xacro:include filename="$(find val_description)/common/xacro/dev_ports/valkyrie_imu_test_ports.xacro"/>

File: model/robots/right_leg.xacro (robot description, xacro)
@@ -6,4 +6,5 @@
     <xacro:include filename="$(find val_description)/common/xacro/api/valkyrie_B_api.xacro"/>
     <xacro:include filename="$(find val_description)/model/robots/common/xacro/leg/link_names.xacro"/>
+    <xacro:include filename="$(find val_description)/common/xacro/nodes/valkyrie_nodes.xacro"/>
     <xacro:property name="prefix" value="right"/>
     <xacro:property name="reflect" value="-1"/>

File: model/robots/valkyrie_A.xacro (robot description, xacro)
@@ -5,4 +5,5 @@
     <xacro:include filename="$(find val_description)/model/robots/common/xacro/valkyrie_base_hw.xacro"/>
     <xacro:include filename="$(find val_description)/common/xacro/serial_numbers/valkyrie_A_serials.xacro"/>
+    <xacro:include filename="$(find val_description)/common/xacro/nodes/valkyrie_nodes.xacro"/>
     <xacro:include filename="$(find val_description)/common/xacro/api/valkyrie_A_api.xacro"/>
     <xacro:include filename="$(find val_description)/common/xacro/dev_ports/valkyrie_A_ports.xacro"/>

File: model/robots/valkyrie_A_arm_mass_sims.xacro (robot description, xacro)
@@ -5,4 +5,5 @@
     <xacro:include filename="$(find val_description)/model/robots/common/xacro/valkyrie_arm_mass_sims_base_hw.xacro"/>
     <xacro:include filename="$(find val_description)/common/xacro/serial_numbers/valkyrie_A_serials.xacro"/>
+    <xacro:include filename="$(find val_description)/common/xacro/nodes/valkyrie_nodes.xacro"/>
     <xacro:include filename="$(find val_description)/common/xacro/api/valkyrie_A_api.xacro"/>
     <xacro:include filename="$(find val_description)/common/xacro/dev_ports/valkyrie_A_ports.xacro"/>

File: model/robots/valkyrie_B.xacro (robot description, xacro)
@@ -5,4 +5,5 @@
     <xacro:include filename="$(find val_description)/model/robots/common/xacro/valkyrie_base_hw.xacro"/>
     <xacro:include filename="$(find val_description)/common/xacro/serial_numbers/valkyrie_B_serials.xacro"/>
+    <xacro:include filename="$(find val_description)/common/xacro/nodes/valkyrie_nodes.xacro"/>
     <xacro:include filename="$(find val_description)/common/xacro/api/valkyrie_B_api.xacro"/>
     <xacro:include filename="$(find val_description)/common/xacro/dev_ports/valkyrie_B_ports.xacro"/>

File: model/robots/valkyrie_B_arm_mass_sims.xacro (robot description, xacro)
@@ -5,4 +5,5 @@
     <xacro:include filename="$(find val_description)/model/robots/common/xacro/valkyrie_arm_mass_sims_base_hw.xacro"/>
     <xacro:include filename="$(find val_description)/common/xacro/serial_numbers/valkyrie_B_serials.xacro"/>
+    <xacro:include filename="$(find val_description)/common/xacro/nodes/valkyrie_nodes.xacro"/>
     <xacro:include filename="$(find val_description)/common/xacro/api/valkyrie_B_api.xacro"/>
     <xacro:include filename="$(find val_description)/common/xacro/dev_ports/valkyrie_B_ports.xacro"/>

File: model/robots/valkyrie_C.xacro (robot description, xacro)
@@ -5,4 +5,5 @@
     <xacro:include filename="$(find val_description)/model/robots/common/xacro/valkyrie_base_hw.xacro"/>
     <xacro:include filename="$(find val_description)/common/xacro/serial_numbers/valkyrie_C_serials.xacro"/>
+    <xacro:include filename="$(find val_description)/common/xacro/nodes/valkyrie_nodes.xacro"/>
     <xacro:include filename="$(find val_description)/common/xacro/api/valkyrie_C_api.xacro"/>
     <xacro:include filename="$(find val_description)/common/xacro/dev_ports/valkyrie_C_ports.xacro"/>

File: model/robots/valkyrie_C_arm_mass_sims.xacro (robot description, xacro)
@@ -5,4 +5,5 @@
     <xacro:include filename="$(find val_description)/model/robots/common/xacro/valkyrie_arm_mass_sims_base_hw.xacro"/>
     <xacro:include filename="$(find val_description)/common/xacro/serial_numbers/valkyrie_C_serials.xacro"/>
+    <xacro:include filename="$(find val_description)/common/xacro/nodes/valkyrie_nodes.xacro"/>
     <xacro:include filename="$(find val_description)/common/xacro/api/valkyrie_C_api.xacro"/>
     <xacro:include filename="$(find val_description)/common/xacro/dev_ports/valkyrie_C_ports.xacro"/>

File: model/robots/valkyrie_D.xacro (robot description, xacro)
@@ -5,4 +5,5 @@
     <xacro:include filename="$(find val_description)/model/robots/common/xacro/valkyrie_base_hw.xacro"/>
     <xacro:include filename="$(find val_description)/common/xacro/serial_numbers/valkyrie_D_serials.xacro"/>
+    <xacro:include filename="$(find val_description)/common/xacro/nodes/valkyrie_nodes.xacro"/>
     <xacro:include filename="$(find val_description)/common/xacro/api/valkyrie_D_api.xacro"/>
     <xacro:include filename="$(find val_description)/common/xacro/dev_ports/valkyrie_D_ports.xacro"/>

File: model/robots/valkyrie_D_arm_mass_sims.xacro (robot description, xacro)
@@ -5,4 +5,5 @@
     <xacro:include filename="$(find val_description)/model/robots/common/xacro/valkyrie_arm_mass_sims_base_hw.xacro"/>
     <xacro:include filename="$(find val_description)/common/xacro/serial_numbers/valkyrie_D_serials.xacro"/>
+    <xacro:include filename="$(find val_description)/common/xacro/nodes/valkyrie_nodes.xacro"/>
     <xacro:include filename="$(find val_description)/common/xacro/api/valkyrie_D_api.xacro"/>
     <xacro:include filename="$(find val_description)/common/xacro/dev_ports/valkyrie_D_ports.xacro"/>

File: model/robots/valkyrie_sim.xacro (robot description, xacro)
@@ -6,4 +6,5 @@
     <xacro:include filename="$(find val_description)/model/urdf/multisense_sl.urdf" />
     <xacro:include filename="$(find val_description)/common/xacro/serial_numbers/valkyrie_A_serials.xacro"/>
+    <xacro:include filename="$(find val_description)/common/xacro/nodes/valkyrie_nodes.xacro"/>
     <xacro:include filename="$(find val_description)/common/xacro/dev_ports/valkyrie_gazebo_ports.xacro"/>
     <xacro:include filename="$(find val_description)/model/robots/common/xacro/valkyrie_base_sim.xacro"/>

File: model/robots/valkyrie_sim_arm_mass_sims.xacro (robot description, xacro)
@@ -6,4 +6,5 @@
     <xacro:include filename="$(find val_description)/model/urdf/multisense_sl.urdf" />
     <xacro:include filename="$(find val_description)/common/xacro/serial_numbers/valkyrie_A_serials.xacro"/>
+    <xacro:include filename="$(find val_description)/common/xacro/nodes/valkyrie_nodes.xacro"/>
     <xacro:include filename="$(find val_description)/common/xacro/dev_ports/valkyrie_gazebo_ports.xacro"/>
     <xacro:include filename="$(find val_description)/model/robots/common/xacro/valkyrie_arm_mass_sims_base_sim.xacro"/>

File: model/robots/valkyrie_sim_pinned.xacro (robot description, xacro)
@@ -7,4 +7,5 @@
     <xacro:include filename="$(find val_description)/model/urdf/multisense_sl.urdf" />
     <xacro:include filename="$(find val_description)/common/xacro/serial_numbers/valkyrie_A_serials.xacro"/>
+    <xacro:include filename="$(find val_description)/common/xacro/nodes/valkyrie_nodes.xacro"/>
     <xacro:include filename="$(find val_description)/common/xacro/dev_ports/valkyrie_gazebo_ports.xacro"/>
     <xacro:include filename="$(find val_description)/common/xacro/api/valkyrie_sim_api.xacro"/>
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