Commit message: corrected error in node file

File: common/xacro/nodes/forearm_new_firmware_test_nodes.xacro (robot description, xacro)
@@ -4,7 +4,7 @@
 	<xacro:property name="IndexFingerPitch1Node" value="/${prefix}_forearm/indexpitch"/>
 	<xacro:property name="MiddleFingerPitch1Node" value="/${prefix}_forearm/middlepitch"/>
-	<xacro:property name="PinkyPitch1Node" value="/${prefix}_forearm//pinkypitch"/>
+	<xacro:property name="PinkyPitch1Node" value="/${prefix}_forearm/pinkypitch"/>
 	<xacro:property name="ThumbRollNode" value="/${prefix}_forearm/thumbroll"/>
-	<xacro:property name="ThumbPitch1Node" value="/${prefix}_forearm/thumbpitch_1"/>
-	<xacro:property name="ThumbPitch2Node" value="/${prefix}_forearm/thumbpitch_2"/>
+	<xacro:property name="ThumbPitch1Node" value="/${prefix}_forearm/thumbpitch1"/>
+	<xacro:property name="ThumbPitch2Node" value="/${prefix}_forearm/thumbpitch2"/>
 </robot>
