Commit message: left forearm with new firmware test working - APS not calibrated

File: common/xacro/serial_numbers/forearm_new_firmware_test_serials.xacro (robot description, xacro)
@@ -1,10 +1,10 @@
 <robot xmlns:xacro="http://ros.org/wiki/xacro" name="forearm_new_firmware_test_serials">
-	<xacro:property name="leftWristBottomActuatorSerialNumber" value="v_a_006" />
-	<xacro:property name="leftWristTopActuatorSerialNumber" value="v_b_002" />
-	<xacro:property name="leftforearmJ1SerialNumber" value="v_c_002" />
-	<xacro:property name="leftforearmJ2SerialNumber" value="v_d_001" />
-	<xacro:property name="leftforearmJ3SerialNumber" value="v_d_001" />
-	<xacro:property name="leftforearmJ4SerialNumber" value="v_d_001" />
-	<xacro:property name="leftforearmJ5SerialNumber" value="v_d_001" />
-	<xacro:property name="leftforearmJ6SerialNumber" value="v_d_001" />
+	<xacro:property name="leftWristBottomActuatorSerialNumber" value="v_h_006" />
+	<xacro:property name="leftWristTopActuatorSerialNumber" value="v_h_008" />
+	<xacro:property name="leftforearmIndexSerialNumber" value="v_h_001" />
+	<xacro:property name="leftforearmMiddleSerialNumber" value="v_h_004" />
+	<xacro:property name="leftforearmPinkySerialNumber" value="v_h_002" />
+	<xacro:property name="leftforearmThumbRollSerialNumber" value="v_h_005" />
+	<xacro:property name="leftforearmThumbPitch1SerialNumber" value="v_h_003" />
+	<xacro:property name="leftforearmThumbPitch2SerialNumber" value="v_h_007" />
 </robot>

File: instance/instances/robots/xacro/common/forearm_new_firmware_template.xacro (robot description, xacro)
@@ -5,7 +5,11 @@
 	<xacro:include filename="$(find val_description)/common/xacro/actuator_names/valkyrie_actuator_names.xacro"/>
 	<RobotInstance id="${instance}" />
-	<xacro:all_channels/>
+        <Channels>
+    		<Channel id="/left_forearm"/>
+	</Channels>
 	<Mechanisms>
-		<xacro:forearm_new_firmware_mechanism prefix="left" forearm_j1_serial_number="${leftforearmJ1SerialNumber}" forearm_j2_serial_number="${leftforearmJ2SerialNumber}" forearm_j3_serial_number="${leftforearmJ3SerialNumber}" forearm_j4_serial_number="${leftforearmJ4SerialNumber}" forearm_j5_serial_number="${leftforearmJ5SerialNumber}" forearm_j6_serial_number="${leftforearmJ6SerialNumber}" wrist_bottom_serial_number="${leftWristBottomActuatorSerialNumber}" wrist_top_serial_number="${leftWristTopActuatorSerialNumber}" />
+		<xacro:forearm_new_firmware_mechanism prefix="left" forearm_index_serial_number="${leftforearmIndexSerialNumber}" forearm_middle_serial_number="${leftforearmMiddleSerialNumber}" forearm_pinky_serial_number="${leftforearmPinkySerialNumber}" forearm_thumbroll_serial_number="${leftforearmThumbRollSerialNumber}" forearm_thumbpitch1_serial_number="${leftforearmThumbPitch1SerialNumber}" forearm_thumbpitch2_serial_number="${leftforearmThumbPitch2SerialNumber}" wrist_bottom_serial_number="${leftWristBottomActuatorSerialNumber}" wrist_top_serial_number="${leftWristTopActuatorSerialNumber}" />
 	</Mechanisms>
+	<Devices>
+	</Devices>
 </robot>

File: instance/instances/robots/xacro/mechanisms/mechanisms.xacro (robot description, xacro)
@@ -33,11 +33,11 @@
     </Mechanism>
 </xacro:macro>
-<xacro:macro name="forearm_new_firmware_mechanism" params="prefix forearm_j1_serial_number forearm_j2_serial_number forearm_j3_serial_number forearm_j4_serial_number forearm_j5_serial_number forearm_j6_serial_number wrist_bottom_serial_number wrist_top_serial_number">
-	<xacro:simple_mechanism name="${IndexFingerPitch1JointName}" serial_number="${forearm_j1_serial_number}" node="${IndexFingerPitch1Node}"/>
-	<xacro:simple_mechanism name="${MiddleFingerPitch1JointName}" serial_number="${forearm_j2_serial_number}" node="${MiddleFingerPitch1Node}"/>
-	<xacro:simple_mechanism name="${PinkyPitch1JointName}" serial_number="${forearm_j3_serial_number}" node="${PinkyPitch1Node}"/>
-	<xacro:simple_mechanism name="${ThumbRollJointName}" serial_number="${forearm_j4_serial_number}" node="${ThumbRollNode}"/>
-	<xacro:simple_mechanism name="${ThumbPitch1JointName}" serial_number="${forearm_j5_serial_number}" node="${ThumbPitch1Node}"/>
-	<xacro:simple_mechanism name="${ThumbPitch2JointName}" serial_number="${forearm_j6_serial_number}" node="${ThumbPitch2Node}"/>
+<xacro:macro name="forearm_new_firmware_mechanism" params="prefix forearm_index_serial_number forearm_middle_serial_number forearm_pinky_serial_number forearm_thumbroll_serial_number forearm_thumbpitch1_serial_number forearm_thumbpitch2_serial_number wrist_bottom_serial_number wrist_top_serial_number">
+	<xacro:simple_mechanism name="${IndexFingerPitch1JointName}" serial_number="${forearm_index_serial_number}" node="${IndexFingerPitch1Node}"/>
+	<xacro:simple_mechanism name="${MiddleFingerPitch1JointName}" serial_number="${forearm_middle_serial_number}" node="${MiddleFingerPitch1Node}"/>
+	<xacro:simple_mechanism name="${PinkyPitch1JointName}" serial_number="${forearm_pinky_serial_number}" node="${PinkyPitch1Node}"/>
+	<xacro:simple_mechanism name="${ThumbRollJointName}" serial_number="${forearm_thumbroll_serial_number}" node="${ThumbRollNode}"/>
+	<xacro:simple_mechanism name="${ThumbPitch1JointName}" serial_number="${forearm_thumbpitch1_serial_number}" node="${ThumbPitch1Node}"/>
+	<xacro:simple_mechanism name="${ThumbPitch2JointName}" serial_number="${forearm_thumbpitch2_serial_number}" node="${ThumbPitch2Node}"/>
 	<xacro:two_active_joint_mechanism mechanism_name="${prefix}Wrist" actuator0_name="${WristBottomActuatorName}" actuator1_name="${WristTopActuatorName}" joint0_name="${WristRollJointName}" joint1_name="${WristPitchJointName}" actuator0_serial="${wrist_bottom_serial_number}" actuator1_serial="${wrist_top_serial_number}" actuator0_node="${WristBottomActuatorNode}" actuator1_node="${WristTopActuatorNode}" />
 </xacro:macro>
