Commit message: updated serial numbers for val B forearm j5's

File: common/xacro/serial_numbers/forearm_left_testbench_serials.xacro (robot description, xacro)
@@ -1,4 +1,4 @@
 <robot xmlns:xacro="http://ros.org/wiki/xacro" name="forearm_testbench">
 	<xacro:property name="forearm_serial_number" value="v_h_007" />
-	<xacro:property name="forearm_yaw_serial_number" value="v_g_016" />
+	<xacro:property name="forearm_yaw_serial_number" value="v_g_021" />
 </robot>

File: common/xacro/serial_numbers/valkyrie_B_serials.xacro (robot description, xacro)
@@ -16,10 +16,10 @@
 	<xacro:property name="leftArmJ3SerialNumber" value="v_f_007" />
 	<xacro:property name="leftArmJ4SerialNumber" value="v_f_008" />
-	<xacro:property name="leftArmJ5SerialNumber" value="v_g_007" />
+	<xacro:property name="leftArmJ5SerialNumber" value="v_g_021" />
 	<xacro:property name="rightArmJ1SerialNumber" value="v_a_010" />
 	<xacro:property name="rightArmJ2SerialNumber" value="v_b_008" />
 	<xacro:property name="rightArmJ3SerialNumber" value="v_f_009" />
 	<xacro:property name="rightArmJ4SerialNumber" value="v_f_010" />
-	<xacro:property name="rightArmJ5SerialNumber" value="v_g_006" />
+	<xacro:property name="rightArmJ5SerialNumber" value="v_g_020" />
 	<xacro:property name="neckJ1SerialNumber" value="v_g_019" />
 	<xacro:property name="neckJ2SerialNumber" value="v_g_010" />
