Commit message: Serial number and coeff change after switching out unit A's left knee.

File: common/xacro/serial_numbers/valkyrie_A_serials.xacro (robot description, xacro)
@@ -3,5 +3,5 @@
 	<xacro:property name="leftLegJ2SerialNumber" value="v_b_002" />
 	<xacro:property name="leftLegJ3SerialNumber" value="v_c_002" />
-	<xacro:property name="leftLegJ4SerialNumber" value="v_d_001" />
+	<xacro:property name="leftLegJ4SerialNumber" value="v_d_005" />
 	<xacro:property name="leftAnkleLeftActuatorSerialNumber" value="v_e_001" />
 	<xacro:property name="leftAnkleRightActuatorSerialNumber" value="v_e_002" />
