Commit message: updated capabilities of imu test urdf to be able to use microstrain imu

File: common/xacro/dev_ports/valkyrie_imu_test_ports.xacro (robot description, xacro)
@@ -1,3 +1,3 @@
 <robot xmlns:xacro="http://ros.org/wiki/xacro" name="valkyrie_imu_test_ports">
-	<xacro:property name="pelvis_middle_imu_port" value="/dev/serial/by-id/usb-FTDI_USB-RS422_Cable_FTVR09ZC-if00-port0" />
+	<xacro:property name="pelvis_middle_imu_port" value="/dev/serial/by-id/usb-MicroStrain__Inc._3DM-GX3-25_Orientation_Sensor_6223.10895______-if00" />
 </robot>

File: model/robots/common/xacro/valkyrie_imu_base.xacro (robot description, xacro)
@@ -1,6 +1,7 @@
 <robot xmlns:xacro="http://ros.org/wiki/xacro" name="valkyrie">
     <xacro:property name="KVHHardwareApi" value="val_imu_kvh_1750_interface/ImuKVHInterface" />
+    <xacro:property name="ImuMicrostrainHardwareApi" value="val_imu_3dm_gx4_15_interface/Imu3dmGx415Interface" />
     <xacro:make_pelvis />
     <xacro:include_multisense_hw />
-    <xacro:v1_pelvis_middle_sensors_usb sensor_node_tag="${pelvis_middle_imu_node}" sensor_api_tag="${KVHHardwareApi}"  sensor_port_tag="${pelvis_middle_imu_port}" sensor_number_tag="3dmConfigTest"/>
+    <xacro:v1_pelvis_middle_sensors_usb sensor_node_tag="${pelvis_middle_imu_node}" sensor_api_tag="${ImuMicrostrainHardwareApi}"  sensor_port_tag="${pelvis_middle_imu_port}" sensor_number_tag="3dmConfigTest"/>
 </robot>

Commit message: updated imu urdf for different imu tests

File: common/xacro/dev_ports/valkyrie_imu_test_ports.xacro (robot description, xacro)
@@ -1,3 +1,4 @@
 <robot xmlns:xacro="http://ros.org/wiki/xacro" name="valkyrie_imu_test_ports">
-	<xacro:property name="pelvis_middle_imu_port" value="/dev/serial/by-id/usb-FTDI_USB-RS422_Cable_FTVR09ZC-if00-port0" />
+	<!--<xacro:property name="pelvis_middle_imu_port" value="/dev/serial/by-id/usb-MEV_USB_RS485_Serial_Converter_Rev4_MVYPUTBJ-if00-port0" /> -->
+	<xacro:property name="pelvis_middle_imu_port" value="/dev/serial/by-id/usb-FTDI_USB-RS422_Cable_FTXRO1OW-if00-port0" />
 </robot>

File: model/robots/common/xacro/valkyrie_imu_base.xacro (robot description, xacro)
@@ -1,6 +1,6 @@
 <robot xmlns:xacro="http://ros.org/wiki/xacro" name="valkyrie">
-    <xacro:property name="KVHHardwareApi" value="val_imu_kvh_1750_interface/ImuKVHInterface" />
+    <xacro:property name="DMUHardwareApi" value="val_imu_kvh_1750_interface/ImuKVHInterface" />
     <xacro:make_pelvis />
     <xacro:include_multisense_hw />
-    <xacro:v1_pelvis_middle_sensors_usb sensor_node_tag="${pelvis_middle_imu_node}" sensor_api_tag="${KVHHardwareApi}"  sensor_port_tag="${pelvis_middle_imu_port}"/>
+    <xacro:v1_pelvis_middle_sensors_usb sensor_node_tag="${pelvis_middle_imu_node}" sensor_api_tag="${DMUHardwareApi}"  sensor_port_tag="${pelvis_middle_imu_port}"/>
 </robot>

Commit message: updating coeffs for unit e arm etc.

File: common/xacro/dev_ports/valkyrie_imu_test_ports.xacro (robot description, xacro)
@@ -1,3 +1,3 @@
 <robot xmlns:xacro="http://ros.org/wiki/xacro" name="valkyrie_imu_test_ports">
-	<xacro:property name="pelvis_middle_imu_port" value="/dev/serial/by-id/usb-FTDI_USB-RS422_Cable_FTVR09ZC-if00-port0" />
+	<xacro:property name="pelvis_middle_imu_port" value="/dev/serial/by-id/usb-Lord_Microstrain_Lord_Inertial_Sensor_0000__6233.47087-if00" />
 </robot>

File: model/robots/common/xacro/valkyrie_imu_base.xacro (robot description, xacro)
@@ -1,4 +1,4 @@
 <robot xmlns:xacro="http://ros.org/wiki/xacro" name="valkyrie">
-    <xacro:property name="KVHHardwareApi" value="val_imu_kvh_1750_interface/ImuKVHInterface" />
+    <xacro:property name="KVHHardwareApi" value="val_imu_3dm_gx4_15_interface/Imu3dmGx415Interface" />
     <xacro:make_pelvis />
     <xacro:include_multisense_hw />
