Commit message: Added non-zero PID gains for the ForearmYaw joint.

File: model/robots/common/xacro/arm/arm.xacro (robot description, xacro)
@@ -121,5 +121,5 @@
                           damping="0.1" friction="0.0">
         <limit effort="${ForearmYawTorqueLimit}" lower="${ForearmYawPositionLimit_Lower}" upper="${ForearmYawPositionLimit_Upper}" velocity="${ForearmYawVelocityLimit}"/>
-        <controller_gains Kp="0.0" Kd="0" Ki="0.0"/>
+        <controller_gains Kp="${ForearmYawKp}" Kd="${ForearmYawKd}" Ki="${ForearmYawKi}"/>
     </xacro:revolute_joint_ex>
     <xacro:revolute_joint_ex jointName="${WristRollJointName}"

File: model/robots/common/xacro/gains.xacro (robot description, xacro)
@@ -1,3 +1,6 @@
 <robot xmlns:xacro="http://ros.org/wiki/xacro" name="valkyrie_nodes">
+    <xacro:property name="ForearmYawKp" value="20000" />
+    <xacro:property name="ForearmYawKd" value="400" />
+    <xacro:property name="ForearmYawKi" value="0.0" />
     <xacro:property name="WristPitchKp" value="20000" />
     <xacro:property name="WristPitchKd" value="400" />
