Commit message: Updated IMU API names based on new names from the refactor.

File: common/xacro/api/valkyrie_A_api.xacro (robot description, xacro)
@@ -20,5 +20,5 @@
     <xacro:property name="WaistRightActuatorApi" value="robot_hardware_interface/TurbodriverAPI_linear_futek" />
     <xacro:property name="AtiSensorApi" value="TurbodriverForceTorqueSensor" />
-    <xacro:property name="ImuMicrostrainHardwareApi" value="val_imu_3dm_gx4_15_interface/Imu3dmGx415Interface" />
+    <xacro:property name="ImuMicrostrainHardwareApi" value="imu_3dm_gx4_15_sensor::Imu3DmGx415Sensor" />
     <xacro:property name="ImuVectorNavHardwareApi" value="val_imu_vectornav_vn100_interface/ImuVecotNavInterface" />
     <xacro:property name="ImuSensorSimApi" value="val_imu_gazebo_interface/ImuGazeboInterface" />

File: common/xacro/api/valkyrie_B_api.xacro (robot description, xacro)
@@ -20,5 +20,5 @@
     <xacro:property name="WaistRightActuatorApi" value="robot_hardware_interface/TurbodriverAPI_linear_Renishaw" />
     <xacro:property name="AtiSensorApi" value="TurbodriverForceTorqueSensor" />
-    <xacro:property name="ImuMicrostrainHardwareApi" value="val_imu_3dm_gx4_15_interface/Imu3dmGx415Interface" />
+    <xacro:property name="ImuMicrostrainHardwareApi" value="imu_3dm_gx4_15_sensor::Imu3DmGx415Sensor" />
     <xacro:property name="ImuVectorNavHardwareApi" value="val_imu_vectornav_vn100_interface/ImuVecotNavInterface" />
     <xacro:property name="ImuSensorSimApi" value="val_imu_gazebo_interface/ImuGazeboInterface" />

File: common/xacro/api/valkyrie_C_api.xacro (robot description, xacro)
@@ -20,5 +20,5 @@
     <xacro:property name="WaistRightActuatorApi" value="robot_hardware_interface/TurbodriverAPI_linear_Renishaw" />
     <xacro:property name="AtiSensorApi" value="TurbodriverForceTorqueSensor" />
-    <xacro:property name="ImuMicrostrainHardwareApi" value="val_imu_3dm_gx4_15_interface/Imu3dmGx415Interface" />
+    <xacro:property name="ImuMicrostrainHardwareApi" value="imu_3dm_gx4_15_sensor::Imu3DmGx415Sensor" />
     <xacro:property name="ImuVectorNavHardwareApi" value="val_imu_vectornav_vn100_interface/ImuVecotNavInterface" />
     <xacro:property name="ImuSensorSimApi" value="val_imu_gazebo_interface/ImuGazeboInterface" />

File: common/xacro/api/valkyrie_sim_api.xacro (robot description, xacro)
@@ -1,5 +1,5 @@
 <robot xmlns:xacro="http://ros.org/wiki/xacro" name="valkyrie_sim_api">
 	<xacro:property name="SimApi" value="robot_hardware_interface/TurbodriverSimAPI" />
-    <xacro:property name="ImuSensorSimApi" value="val_imu_gazebo_interface/ImuGazeboInterface" />
+    <xacro:property name="ImuSensorSimApi" value="simulated_imu_sensor::SimulatedImuSensor" />
     <xacro:property name="AtiSensorApi" value="TurbodriverForceTorqueSensor" />
 </robot>
